Commit message: Update localization and vehicle configuration

File: ros2_ws/src/vehicle_description/urdf/rc_car.urdf.xacro (robot description, xacro)
@@ -141,5 +141,5 @@
     <parent link="base_link"/>
     <child link="imu_link"/>
-    <origin xyz="${wheel_base + imu_dx} 0 ${ground_clearance + chassis_height - wheel_radius}" rpy="0 0 0"/>
+    <origin xyz="${wheel_base + imu_dx} 0 ${ground_clearance + chassis_height - wheel_radius}" rpy="0 0 ${-pi/2}"/>
   </joint>
   <!-- GPS: position barely matters at this accuracy, so it sits on top of the chassis centre -->

Commit message: Lidar integration

File: ros2_ws/src/vehicle_description/urdf/rc_car.urdf.xacro (robot description, xacro)
@@ -150,3 +150,10 @@
     <origin xyz="0 0 ${chassis_height/2}" rpy="0 0 0"/>
   </joint>
+  <!-- RPLIDAR A1M8 at the chassis centreline and top surface. -->
+  <link name="lidar_link"/>
+  <joint name="lidar_joint" type="fixed">
+    <parent link="base_link"/>
+    <child link="lidar_link"/>
+    <origin xyz="${chassis_x_offset} 0 ${ground_clearance + chassis_height - wheel_radius}" rpy="0 0 0"/>
+  </joint>
 </robot>
