Commit message: Replace RC description with ENIMIA and add simulation package

File: ros2_ws/src/vehicle_description/urdf/enimia.urdf (robot description, URDF)
Before this commit: robot enimia_black, 11 links, 10 joints
Links:
- link body_link: geometry collision mesh filename=package://vehicle_description/meshes/body_collision.stl; visual mesh filename=package://vehicle_description/meshes/body_shell.dae

Commit message: Add simulation world and update vehicle model

File: ros2_ws/src/vehicle_description/urdf/enimia.urdf (robot description, URDF)
Before this commit: robot enimia_black, 11 links, 10 joints
Links:
- added link sensor_mount_link, mass 0.2; visual box size=0.30 0.20 0.006; visual cylinder length=0.054 radius=0.012
- link gps_link: mass None -> 0.03; geometry visual box size=0.03 0.03 0.01
- link imu_link: mass None -> 0.005; geometry visual box size=0.027 0.020 0.004
- link lidar_link: mass None -> 0.17; geometry visual cylinder length=0.041 radius=0.0355
Joints:
- added joint sensor_mount_joint: type fixed, parent base_link, child sensor_mount_link, origin xyz=0.050 0.000 0.492 rpy=0 0 0
- joint gps_joint: origin xyz=-0.100 0.000 0.455 rpy=0 0 0 -> xyz=-0.100 0.000 0.010 rpy=0 0 0; parent base_link -> sensor_mount_link
- joint imu_joint: origin xyz=0.000 0.000 0.060 rpy=0 0 0 -> xyz=0.070 0.070 0.000 rpy=0 0 0; parent base_link -> sensor_mount_link
- joint lidar_joint: origin xyz=0.100 0.000 0.445 rpy=0 0.139626 0 -> xyz=0.070 0.000 0.075 rpy=0 0.139626 0; parent base_link -> sensor_mount_link

Commit message: Update simulation and Silesia Ring world

File: ros2_ws/src/vehicle_description/urdf/enimia.urdf (robot description, URDF)
Before this commit: robot enimia_black, 12 links, 11 joints
Joints:
- joint lidar_joint: origin xyz=0.070 0.000 0.075 rpy=0 0.139626 0 -> xyz=0.070 0.000 0.075 rpy=0 0.07 0
